Commit message: Removed ros2_control from sim interface

File: smart_diffbot_description/model/urdf/sim_interface.urdf.xacro (robot description, xacro)
@@ -1,32 +1,6 @@
 <?xml version="1.0"?>
 <robot xmlns:xacro="http://ros.org/wiki/xacro">
-  <!-- Simulation ros2_control interface -->
-  <ros2_control name="IgnitionSystem" type="system">
-    <hardware>
-      <plugin>ign_ros2_control/IgnitionSystem</plugin>
-    </hardware>
-    <joint name="left_wheel_joint">
-      <command_interface name="velocity">
-        <param name="min">-10</param>
-        <param name="max">10</param>
-      </command_interface>
-      <state_interface name="position"/>
-      <state_interface name="velocity"/>
-    </joint>
-    <joint name="right_wheel_joint">
-      <command_interface name="velocity">
-        <param name="min">-10</param>
-        <param name="max">10</param>
-      </command_interface>
-      <state_interface name="position"/>
-      <state_interface name="velocity"/>
-    </joint>
-  </ros2_control>
    <!-- Gazebo plugins -->
    <gazebo>
-    <!-- ros2_control -->
-    <plugin filename="ign_ros2_control-system" name="ign_ros2_control::IgnitionROS2ControlPlugin">
-      <parameters>$(find smart_diffbot_control)/config/controller_params.yaml</parameters>
-    </plugin>
     <!-- sensors -->
     <plugin filename="ignition-gazebo-sensors-system"  name="ignition::gazebo::systems::Sensors">

Commit message: update simulation interface

File: smart_diffbot_description/model/urdf/sim_interface.urdf.xacro (robot description, xacro)
@@ -22,4 +22,19 @@
       <state_interface name="velocity"/>
     </joint>
+    <joint name="camera_base_joint">
+      <command_interface name="position"/>
+      <state_interface name="position"/>
+      <state_interface name="velocity"/>
+    </joint>
+    <joint name="camera_link_joint">
+      <command_interface name="position"/>
+      <state_interface name="position"/>
+      <state_interface name="velocity"/>
+    </joint>
+    <joint name="camera_top_joint">
+      <command_interface name="position"/>
+      <state_interface name="position"/>
+      <state_interface name="velocity"/>
+    </joint>
   </ros2_control>
    <!-- Gazebo plugins -->
@@ -39,5 +54,5 @@
   </gazebo>
   <!-- Sensor simulation -->
-  <gazebo reference="camera_link">
+  <gazebo reference="sensor_link">
     <sensor name="camera" type="camera">
       <always_on>1</always_on>
@@ -45,5 +60,5 @@
       <visualize>true</visualize>
       <topic>camera/image_raw</topic>
-      <ignition_frame_id>camera_link</ignition_frame_id>
+      <ignition_frame_id>sensor_link</ignition_frame_id>
     </sensor>
   </gazebo>
