Commit message: update hardware xacro for wheel motor numbering

File: smart_diffbot_description/model/urdf/hardware.urdf.xacro (robot description, xacro)
@@ -7,7 +7,8 @@
       <param name="usb_port">/dev/ttyUSB0</param>
       <param name="baud_rate">1000000</param>
+      <!-- <param name="use_dummy">true</param> -->
     </hardware>
-    <joint name="left_wheel_joint">
-      <param name="id">11</param>
+    <joint name="right_wheel_joint">
+      <param name="id">1</param>
       <command_interface name="position"/>
       <command_interface name="velocity">
@@ -18,6 +19,6 @@
       <state_interface name="velocity"/>
     </joint>
-    <joint name="right_wheel_joint">
-      <param name="id">12</param>
+    <joint name="left_wheel_joint">
+      <param name="id">2</param>
       <command_interface name="position"/>
       <command_interface name="velocity">

Commit message: add mock system for camera joints

File: smart_diffbot_description/model/urdf/hardware.urdf.xacro (robot description, xacro)
@@ -1,5 +1,5 @@
 <?xml version="1.0"?>
 <robot xmlns:xacro="http://ros.org/wiki/xacro">
-  <!-- Simulation ros2_control interface -->
+  <!-- Dynamixel ros2_control interface -->
   <ros2_control name="DynamixelSystem" type="system">
     <hardware>
@@ -30,3 +30,27 @@
     </joint>
   </ros2_control>
+    <!-- Camera ros2_control interface -->
+  <ros2_control name="CameraSystem" type="system">
+    <hardware>
+      <plugin>mock_components/GenericSystem</plugin>
+    </hardware>
+    <joint name="camera_base_joint">
+      <command_interface name="position"/>
+      <command_interface name="velocity"/>
+      <state_interface name="position"/>
+      <state_interface name="velocity"/>
+    </joint>
+    <joint name="camera_link_joint">
+      <command_interface name="position"/>
+      <command_interface name="velocity"/>
+      <state_interface name="position"/>
+      <state_interface name="velocity"/>
+    </joint>
+    <joint name="camera_top_joint">
+      <command_interface name="position"/>
+      <command_interface name="velocity"/>
+      <state_interface name="position"/>
+      <state_interface name="velocity"/>
+    </joint>
+  </ros2_control>
 </robot>
