Commit message: update robot dimensions to match actual hardware

File: smart_diffbot_description/model/urdf/camera.urdf.xacro (robot description, xacro)
@@ -1,14 +1,14 @@
 <?xml version="1.0"?>
 <robot xmlns:xacro="http://ros.org/wiki/xacro">
-  <xacro:property name="camera_link_width" value="0.02"/>
-  <xacro:property name="camera_link_depth" value="0.05"/>
-  <xacro:property name="camera_length" value="0.25"/>
-  <xacro:property name="camera_height" value="0.1"/>
-  <xacro:property name="camera_base_height" value="0.05"/>
-  <xacro:property name="camera_offset" value="0.05"/>
-  <xacro:property name="camera_radius" value="0.1"/>
-  <xacro:property name="camera_link_length" value="0.3"/>
-  <xacro:property name="lens_radius" value="0.04"/>
-  <xacro:property name="lens_length" value="0.02"/>
+  <xacro:property name="camera_link_width" value="0.002"/>
+  <xacro:property name="camera_link_depth" value="0.005"/>
+  <xacro:property name="camera_length" value="0.025"/>
+  <xacro:property name="camera_height" value="0.01"/>
+  <xacro:property name="camera_base_height" value="0.005"/>
+  <xacro:property name="camera_offset" value="0.005"/>
+  <xacro:property name="camera_radius" value="0.01"/>
+  <xacro:property name="camera_link_length" value="0.03"/>
+  <xacro:property name="lens_radius" value="0.004"/>
+  <xacro:property name="lens_length" value="0.002"/>
   <!-- Wheel macro -->
   <xacro:macro name="camera" params="name parent">

File: smart_diffbot_description/model/urdf/model.urdf.xacro (robot description, xacro)
@@ -4,12 +4,12 @@
   <xacro:include filename="$(find smart_diffbot_description)/model/urdf/camera.urdf.xacro" />
   <!-- Properties -->
-  <xacro:property name="base_length" value="1.5"/>
-  <xacro:property name="base_width" value="1.0"/>
-  <xacro:property name="base_height" value="0.5"/>
-  <xacro:property name="wheel_radius" value="0.2"/>
-  <xacro:property name="wheel_width" value="0.1"/>
-  <xacro:property name="wheel_suspension" value="0.05"/>
-  <xacro:property name="wheel_spacing" value="0.02"/>
-  <xacro:property name="caster_radius" value="0.07"/>
+  <xacro:property name="base_length" value="0.1415"/>
+  <xacro:property name="base_width" value="0.09"/>
+  <xacro:property name="base_height" value="0.07"/>
+  <xacro:property name="wheel_radius" value="0.033"/>
+  <xacro:property name="wheel_width" value="0.018"/>
+  <xacro:property name="wheel_suspension" value="0.01"/>
+  <xacro:property name="wheel_spacing" value="0.002"/>
+  <xacro:property name="caster_radius" value="0.015"/>
   <!-- Links -->
   <link name="base_link">
@@ -54,5 +54,5 @@
       </geometry>
     </collision>
-    <xacro:box_inertia m="0.5" w="${base_width}" d="${base_length}" h="${base_height}"/>
+    <xacro:sphere_inertia m="0.25" r="${caster_radius}"/>
   </link>
   <!-- Joints -->

Commit message: fix camera collision model

File: smart_diffbot_description/model/urdf/camera.urdf.xacro (robot description, xacro)
@@ -40,5 +40,5 @@
       </visual>
       <collision>
-        <origin xyz="0 0 0" rpy="0 0 0"/>
+        <origin xyz="0 0 0" rpy="0 ${pi/2} 0"/>
         <geometry>
           <cylinder radius="${lens_radius}" length="${lens_length}" />
@@ -67,5 +67,5 @@
     </link>
     <!-- Camera link -->
-      <link name="${name}_link">
+    <link name="${name}_link">
       <visual>
         <origin xyz="0 ${camera_radius+camera_link_width/2.0} ${camera_link_length/2.0}" rpy="0 0 0"/>
@@ -83,8 +83,16 @@
       </visual>
       <collision>
-        <origin xyz="0 ${camera_radius*2.0+camera_link_width/2.0} ${camera_link_length/2.0}" rpy="0 0 0"/>
+        <origin xyz="0 ${camera_radius+camera_link_width/2.0} ${camera_link_length/2.0}" rpy="0 0 0"/>
         <geometry>
           <box size="${camera_link_depth} ${camera_link_width} ${camera_link_length}" />
         </geometry>
+        <material name="white"/>
+      </collision>
+      <collision>
+        <origin xyz="0 -${camera_radius+camera_link_width/2.0} ${camera_link_length/2.0}" rpy="0 0 0"/>
+        <geometry>
+          <box size="${camera_link_depth} ${camera_link_width} ${camera_link_length}" />
+        </geometry>
+        <material name="white"/>
       </collision>
       <xacro:box_inertia m="1.0" w="${camera_link_depth}" d="${camera_link_width}" h="${camera_link_length}"/>
