Commit message: add _bringup and _description updates from final branch

File: smart_diffbot_description/model/urdf/robot.urdf.xacro (robot description, xacro)
@@ -1,5 +1,4 @@
 <?xml version="1.0"?>
 <robot name="smart_diffbot" xmlns:xacro="http://ros.org/wiki/xacro">
-  <!-- Arguments -->
   <xacro:arg name="sim" default="true"/>
   <!-- Utils -->
@@ -7,10 +6,10 @@
   <!-- Robot model -->
   <xacro:include filename="$(find smart_diffbot_description)/model/urdf/model.urdf.xacro" />
-  <!-- Simulation interface -->
   <xacro:if value="$(arg sim)">
+    <!-- Simulation interface -->
     <xacro:include filename="$(find smart_diffbot_description)/model/urdf/sim_interface.urdf.xacro" />
   </xacro:if>
-  <!-- Hardware interface -->
   <xacro:unless value="$(arg sim)">
+    <!-- Real hardware -->
     <xacro:include filename="$(find smart_diffbot_description)/model/urdf/hardware.urdf.xacro" />
   </xacro:unless>

File: smart_diffbot_description/model/urdf/sim_interface.urdf.xacro (robot description, xacro)
@@ -1,17 +1,61 @@
 <?xml version="1.0"?>
 <robot xmlns:xacro="http://ros.org/wiki/xacro">
+  <!-- Simulation ros2_control interface -->
+  <ros2_control name="GazeboSystem" type="system">
+    <hardware>
+      <plugin>gz_ros2_control/GazeboSimSystem</plugin>
+    </hardware>
+    <joint name="left_wheel_joint">
+      <command_interface name="velocity">
+        <param name="min">-10</param>
+        <param name="max">10</param>
+      </command_interface>
+      <state_interface name="position"/>
+      <state_interface name="velocity"/>
+    </joint>
+    <joint name="right_wheel_joint">
+      <command_interface name="velocity">
+        <param name="min">-10</param>
+        <param name="max">10</param>
+      </command_interface>
+      <state_interface name="position"/>
+      <state_interface name="velocity"/>
+    </joint>
+    <joint name="camera_base_joint">
+      <command_interface name="position"/>
+      <command_interface name="velocity"/>
+      <state_interface name="position"/>
+      <state_interface name="velocity"/>
+    </joint>
+    <joint name="camera_link_joint">
+      <command_interface name="position"/>
+      <command_interface name="velocity"/>
+      <state_interface name="position"/>
+      <state_interface name="velocity"/>
+    </joint>
+    <joint name="camera_top_joint">
+      <command_interface name="position"/>
+      <command_interface name="velocity"/>
+      <state_interface name="position"/>
+      <state_interface name="velocity"/>
+    </joint>
+  </ros2_control>
    <!-- Gazebo plugins -->
    <gazebo>
+    <!-- ros2_control -->
+    <plugin filename="gz_ros2_control-system" name="gz_ros2_control::GazeboSimROS2ControlPlugin">
+      <parameters>$(find smart_diffbot_control)/config/controller_params.yaml</parameters>
+    </plugin>
     <!-- sensors -->
-    <plugin filename="ignition-gazebo-sensors-system"  name="ignition::gazebo::systems::Sensors">
+    <plugin filename="gz-sim-sensors-system"  name="gz::sim::systems::Sensors">
       <render_engine>ogre2</render_engine>
     </plugin>
     <!-- navsat -->
-    <plugin filename="ignition-gazebo-navsat-system" name="ignition::gazebo::systems::NavSat"/>
+    <plugin filename="gz-sim-navsat-system" name="gz::sim::systems::NavSat"/>
     <!-- IMU -->
-    <plugin filename="libignition-gazebo-imu-system.so" name="ignition::gazebo::systems::Imu"/>
+    <plugin filename="gz-sim-imu-system" name="gz::sim::systems::Imu"/>
   </gazebo>
   <!-- Sensor simulation -->
-  <gazebo reference="camera_link">
+  <gazebo reference="camera_sensor_link">
     <sensor name="camera" type="camera">
       <always_on>1</always_on>
@@ -19,5 +63,5 @@
       <visualize>true</visualize>
       <topic>camera/image_raw</topic>
-      <ignition_frame_id>camera_link</ignition_frame_id>
+      <gz_frame_id>camera_sensor_link</gz_frame_id>
     </sensor>
   </gazebo>
@@ -27,5 +71,5 @@
       <update_rate>1</update_rate>
       <topic>navsat/fix</topic>
-      <ignition_frame_id>navsat_link</ignition_frame_id>
+      <gz_frame_id>navsat_link</gz_frame_id>
     </sensor>
   </gazebo>
@@ -36,6 +80,6 @@
       <visualize>false</visualize>
       <topic>imu/data</topic>
-      <ignition_frame_id>imu_link</ignition_frame_id>
-  </sensor>
+      <gz_frame_id>navsat_link</gz_frame_id>
+    </sensor>
   </gazebo>
   <!-- No friction on fixed caster wheel -->

Commit message: updates for control exercises

File: smart_diffbot_description/model/urdf/robot.urdf.xacro (robot description, xacro)
@@ -12,5 +12,5 @@
   <xacro:unless value="$(arg sim)">
     <!-- Real hardware -->
-    <xacro:include filename="$(find smart_diffbot_description)/model/urdf/hardware.urdf.xacro" />
+    <xacro:include filename="$(find smart_diffbot_description)/model/urdf/hardware_interface.urdf.xacro" />
   </xacro:unless>
 </robot>

File: smart_diffbot_description/model/urdf/sim_interface.urdf.xacro (robot description, xacro)
@@ -1,50 +1,6 @@
 <?xml version="1.0"?>
 <robot xmlns:xacro="http://ros.org/wiki/xacro">
-  <!-- Simulation ros2_control interface -->
-  <ros2_control name="GazeboSystem" type="system">
-    <hardware>
-      <plugin>gz_ros2_control/GazeboSimSystem</plugin>
-    </hardware>
-    <joint name="left_wheel_joint">
-      <command_interface name="velocity">
-        <param name="min">-10</param>
-        <param name="max">10</param>
-      </command_interface>
-      <state_interface name="position"/>
-      <state_interface name="velocity"/>
-    </joint>
-    <joint name="right_wheel_joint">
-      <command_interface name="velocity">
-        <param name="min">-10</param>
-        <param name="max">10</param>
-      </command_interface>
-      <state_interface name="position"/>
-      <state_interface name="velocity"/>
-    </joint>
-    <joint name="camera_base_joint">
-      <command_interface name="position"/>
-      <command_interface name="velocity"/>
-      <state_interface name="position"/>
-      <state_interface name="velocity"/>
-    </joint>
-    <joint name="camera_link_joint">
-      <command_interface name="position"/>
-      <command_interface name="velocity"/>
-      <state_interface name="position"/>
-      <state_interface name="velocity"/>
-    </joint>
-    <joint name="camera_top_joint">
-      <command_interface name="position"/>
-      <command_interface name="velocity"/>
-      <state_interface name="position"/>
-      <state_interface name="velocity"/>
-    </joint>
-  </ros2_control>
    <!-- Gazebo plugins -->
    <gazebo>
-    <!-- ros2_control -->
-    <plugin filename="gz_ros2_control-system" name="gz_ros2_control::GazeboSimROS2ControlPlugin">
-      <parameters>$(find smart_diffbot_control)/config/controller_params.yaml</parameters>
-    </plugin>
     <!-- sensors -->
     <plugin filename="gz-sim-sensors-system"  name="gz::sim::systems::Sensors">
