Commit message: updates for interfacing actual hardware

File: smart_diffbot_description/model/urdf/hardware_interface.urdf.xacro (robot description, xacro)
@@ -4,12 +4,14 @@
   <ros2_control name="DynamixelSystem" type="system">
     <hardware>
-      <plugin>dynamixel_hardware/DynamixelHardware</plugin>
+      <plugin>dynamixel_hw/DynamixelHw</plugin>
       <param name="usb_port">/dev/ttyUSB0</param>
       <param name="baud_rate">1000000</param>
+      <param name="left_wheel_name">left_wheel_joint</param>
+      <param name="right_wheel_name">right_wheel_joint</param>
       <!-- <param name="use_dummy">true</param> -->
     </hardware>
     <joint name="right_wheel_joint">
       <param name="id">1</param>
-      <command_interface name="position"/>
+      <param name="invert">true</param>
       <command_interface name="velocity">
         <param name="min">-10</param>
@@ -21,5 +23,5 @@
     <joint name="left_wheel_joint">
       <param name="id">2</param>
-      <command_interface name="position"/>
+      <param name="invert">false</param>
       <command_interface name="velocity">
         <param name="min">-10</param>

File: smart_diffbot_description/model/urdf/model.urdf.xacro (robot description, xacro)
@@ -31,5 +31,4 @@
     <xacro:box_inertia m="30.0" w="${base_width}" d="${base_length}" h="${base_height}"/>
   </link>
-  <link name="base_footprint"/>
   <link name="camera_mount"/>
   <xacro:camera name="camera" parent="camera_mount"/>
