Commit message: Removed contents of camera model

File: smart_diffbot_description/model/urdf/model.urdf.xacro (robot description, xacro)
@@ -33,26 +33,24 @@
   <!-- Start of camera on top of smart_diffbot -->
   <!--                                         -->
-  <xacro:property name="camera_width" value="0.2"/>
-  <xacro:property name="camera_depth" value="0.05"/>
-  <xacro:property name="camera_height" value="0.1"/>
-  <xacro:property name="lens_radius" value="0.03"/>
-  <xacro:property name="lens_length" value="0.02"/>
+  <xacro:property name="camera_width" value="0.0"/>
+  <xacro:property name="camera_depth" value="0.0"/>
+  <xacro:property name="camera_height" value="0.0"/>
+  <xacro:property name="lens_radius" value="0.0"/>
+  <xacro:property name="lens_length" value="0.0"/>
   <!-- Camera body -->
   <link name="camera_body_link">
     <visual>
-      <origin xyz="0 0 0" rpy="0 0 0"/>
       <geometry>
-        <box size="${camera_depth} ${camera_width} ${camera_height}" />
+        <!-- Insert camera body shape -->
       </geometry>
-      <material name="black" />
-    </visual>
+        <!-- Insert camera body color -->
+      </visual>
     <collision>
-      <origin xyz="0 0 0" rpy="0 0 0"/>
       <geometry>
-        <box size="${camera_depth} ${camera_width} ${camera_height}" />
+        <!-- Insert camera body shape -->
       </geometry>
     </collision>
-    <xacro:box_inertia m="1.0" w="${camera_width}" d="${camera_depth}" h="${camera_height}"/>
-  </link>
+        <!-- Insert camera body inertia -->
+    </link>
   <!-- Camera lens -->
   <link name="camera_lens_link">
@@ -60,31 +58,24 @@
       <origin xyz="0 0 0" rpy="0 ${pi/2} 0"/>
       <geometry>
-        <cylinder radius="${lens_radius}" length="${lens_length}" />
+        <!-- Insert camera lens shape -->
       </geometry>
-      <material name="white" />
+      <!-- Insert camera lens color -->
     </visual>
     <collision>
-      <origin xyz="0 0 0" rpy="0 0 0"/>
       <geometry>
-        <cylinder radius="${lens_radius}" length="${lens_length}" />
+        <!-- Insert camera lens shape -->
       </geometry>
     </collision>
-    <xacro:cylinder_inertia m="0.1" r="${lens_radius}" h="${lens_length}"/>
+        <!-- Insert camera lens inertia -->
   </link>
-  <!-- Camera sensor link -->
-  <link name="camera_link"/>
-  <!-- Camera joints -->
-  <joint name="camera_sensor_joint" type="fixed">
-    <origin xyz="${lens_length/2.0 + 0.1} 0 0" rpy="0 0 0"/>
-    <parent link="camera_lens_link"/>
-    <child link="camera_link"/>
-  </joint>
+  <!-- Joint connecting camera lens to camera body -->
   <joint name="camera_lens_joint" type="fixed">
-    <origin xyz="${camera_depth/2.0} 0 0" rpy="0 0 0"/>
+    <origin xyz="0 0 0" rpy="0 0 0"/>
     <parent link="camera_body_link"/>
     <child link="camera_lens_link"/>
   </joint>
+  <!-- Joint connecting camera body to robot base_link -->
   <joint name="camera_body_joint" type="fixed">
-    <origin xyz="${base_length/2.0 - camera_depth/2.0} 0 ${base_height/2.0 + camera_height/2.0}" rpy="0 0 0"/>
+    <origin xyz="0 0 0" rpy="0 0 0"/>
     <parent link="base_link"/>
     <child link="camera_body_link"/>
@@ -96,4 +87,5 @@
   <link name="imu_link"/>
   <link name="navsat_link"/>
+  <link name="camera_link"/>
   <!-- Wheel links -->
   <xacro:wheel name="left_wheel" width="${wheel_width}" radius="${wheel_radius}" mass="1.0" color="white"/>
@@ -131,4 +123,9 @@
     <child link="navsat_link"/>
   </joint>
+  <joint name="camera_sensor_joint" type="fixed">
+    <origin xyz="${lens_length/2.0 + 0.1} 0 0" rpy="0 0 0"/>
+    <parent link="camera_lens_link"/>
+    <child link="camera_link"/>
+  </joint>
   <joint name="left_wheel_joint" type="continuous">
     <parent link="base_link"/>

Commit message: Cleanup of URDF

File: smart_diffbot_description/model/urdf/model.urdf.xacro (robot description, xacro)
@@ -34,5 +34,5 @@
   <!--                                         -->
   <xacro:property name="camera_width" value="0.0"/>
-  <xacro:property name="camera_depth" value="0.0"/>
+  <xacro:property name="camera_length" value="0.0"/>
   <xacro:property name="camera_height" value="0.0"/>
   <xacro:property name="lens_radius" value="0.0"/>
@@ -51,6 +51,6 @@
       </geometry>
     </collision>
-        <!-- Insert camera body inertia -->
-    </link>
+    <!-- Insert camera body inertia -->
+  </link>
   <!-- Camera lens -->
   <link name="camera_lens_link">
@@ -67,9 +67,9 @@
       </geometry>
     </collision>
-        <!-- Insert camera lens inertia -->
+    <!-- Insert camera lens inertia -->
   </link>
   <!-- Joint connecting camera lens to camera body -->
   <joint name="camera_lens_joint" type="fixed">
-    <origin xyz="0 0 0" rpy="0 0 0"/>
+    <origin xyz="1 0 0" rpy="0 0 0"/>
     <parent link="camera_body_link"/>
     <child link="camera_lens_link"/>
@@ -77,5 +77,5 @@
   <!-- Joint connecting camera body to robot base_link -->
   <joint name="camera_body_joint" type="fixed">
-    <origin xyz="0 0 0" rpy="0 0 0"/>
+    <origin xyz="0 0 1" rpy="0 0 0"/>
     <parent link="base_link"/>
     <child link="camera_body_link"/>

Commit message: update model properties to match hardware version

File: smart_diffbot_description/model/urdf/model.urdf.xacro (robot description, xacro)
@@ -2,12 +2,12 @@
 <robot xmlns:xacro="http://ros.org/wiki/xacro">
   <!-- Properties -->
-  <xacro:property name="base_length" value="1.5"/>
-  <xacro:property name="base_width" value="1.0"/>
-  <xacro:property name="base_height" value="0.5"/>
-  <xacro:property name="wheel_radius" value="0.2"/>
-  <xacro:property name="wheel_width" value="0.1"/>
-  <xacro:property name="wheel_suspension" value="0.05"/>
-  <xacro:property name="wheel_spacing" value="0.02"/>
-  <xacro:property name="caster_radius" value="0.07"/>
+  <xacro:property name="base_length" value="0.1415"/>
+  <xacro:property name="base_width" value="0.09"/>
+  <xacro:property name="base_height" value="0.07"/>
+  <xacro:property name="wheel_radius" value="0.033"/>
+  <xacro:property name="wheel_width" value="0.018"/>
+  <xacro:property name="wheel_suspension" value="0.01"/>
+  <xacro:property name="wheel_spacing" value="0.002"/>
+  <xacro:property name="caster_radius" value="0.01"/>
   <!-- Links -->
   <link name="base_link">

Commit message: update diffbot dimensions to match actual hardware

File: smart_diffbot_description/model/urdf/model.urdf.xacro (robot description, xacro)
@@ -2,12 +2,12 @@
 <robot xmlns:xacro="http://ros.org/wiki/xacro">
   <!-- Properties -->
-  <xacro:property name="base_length" value="1.5"/>
-  <xacro:property name="base_width" value="1.0"/>
-  <xacro:property name="base_height" value="0.5"/>
-  <xacro:property name="wheel_radius" value="0.2"/>
-  <xacro:property name="wheel_width" value="0.1"/>
-  <xacro:property name="wheel_suspension" value="0.05"/>
-  <xacro:property name="wheel_spacing" value="0.02"/>
-  <xacro:property name="caster_radius" value="0.07"/>
+  <xacro:property name="base_length" value="0.1415"/>
+  <xacro:property name="base_width" value="0.09"/>
+  <xacro:property name="base_height" value="0.07"/>
+  <xacro:property name="wheel_radius" value="0.033"/>
+  <xacro:property name="wheel_width" value="0.018"/>
+  <xacro:property name="wheel_suspension" value="0.01"/>
+  <xacro:property name="wheel_spacing" value="0.002"/>
+  <xacro:property name="caster_radius" value="0.01"/>
   <!-- Links -->
   <link name="base_link">
@@ -33,9 +33,9 @@
   <!-- Start of camera on top of smart_diffbot -->
   <!--                                         -->
-  <xacro:property name="camera_width" value="0.2"/>
-  <xacro:property name="camera_depth" value="0.05"/>
-  <xacro:property name="camera_height" value="0.1"/>
-  <xacro:property name="lens_radius" value="0.03"/>
-  <xacro:property name="lens_length" value="0.02"/>
+  <xacro:property name="camera_width" value="0.02"/>
+  <xacro:property name="camera_depth" value="0.005"/>
+  <xacro:property name="camera_height" value="0.01"/>
+  <xacro:property name="lens_radius" value="0.003"/>
+  <xacro:property name="lens_length" value="0.002"/>
   <!-- Camera body -->
   <link name="camera_body_link">

Commit message: update URDF with camera attached to links

File: smart_diffbot_description/model/urdf/model.urdf.xacro (robot description, xacro)
@@ -33,25 +33,30 @@
   <!-- Start of camera on top of smart_diffbot -->
   <!--                                         -->
-  <xacro:property name="camera_width" value="0.2"/>
-  <xacro:property name="camera_depth" value="0.05"/>
+  <xacro:property name="camera_link_width" value="0.02"/>
+  <xacro:property name="camera_link_depth" value="0.05"/>
+  <xacro:property name="camera_length" value="0.25"/>
   <xacro:property name="camera_height" value="0.1"/>
-  <xacro:property name="lens_radius" value="0.03"/>
+  <xacro:property name="camera_base_height" value="0.05"/>
+  <xacro:property name="camera_offset" value="0.05"/>
+  <xacro:property name="camera_radius" value="0.075"/>
+  <xacro:property name="camera_link_length" value="0.3"/>
+  <xacro:property name="lens_radius" value="0.04"/>
   <xacro:property name="lens_length" value="0.02"/>
   <!-- Camera body -->
   <link name="camera_body_link">
     <visual>
-      <origin xyz="0 0 0" rpy="0 0 0"/>
-      <geometry>
-        <box size="${camera_depth} ${camera_width} ${camera_height}" />
-      </geometry>
-      <material name="black" />
-    </visual>
-    <collision>
-      <origin xyz="0 0 0" rpy="0 0 0"/>
-      <geometry>
-        <box size="${camera_depth} ${camera_width} ${camera_height}" />
-      </geometry>
-    </collision>
-    <xacro:box_inertia m="1.0" w="${camera_width}" d="${camera_depth}" h="${camera_height}"/>
+      <origin xyz="${camera_length/4} 0 0" rpy="0 ${pi/2} 0"/>
+      <geometry>
+        <cylinder radius="${camera_radius}" length="${camera_length}"/>
+      </geometry>
+      <material name="white" />
+    </visual>
+    <collision>
+      <origin xyz="0 0 0" rpy="0 0 0"/>
+      <geometry>
+        <cylinder radius="${camera_radius}" length="${camera_length}"/>
+      </geometry>
+    </collision>
+    <xacro:cylinder_inertia m="1.0" r="${camera_radius}" h="${camera_length}"/>
   </link>
   <!-- Camera lens -->
@@ -62,5 +67,5 @@
         <cylinder radius="${lens_radius}" length="${lens_length}" />
       </geometry>
-      <material name="white" />
+      <material name="black" />
     </visual>
     <collision>
@@ -73,20 +78,77 @@
   </link>
   <!-- Camera sensor link -->
-  <link name="camera_link"/>
+  <link name="sensor_link"/>
+    <!-- Camera base -->
+  <link name="camera_base">
+    <visual>
+      <origin xyz="0 0 ${camera_base_height/2}" rpy="0 0 0"/>
+      <geometry>
+        <cylinder radius="${camera_radius}" length="${camera_height}" />
+      </geometry>
+      <material name="SaxionGreen" />
+    </visual>
+    <collision>
+      <origin xyz="0 0 ${camera_base_height/2}" rpy="0 0 0"/>
+      <geometry>
+        <cylinder radius="${camera_radius}" length="${camera_height}" />
+      </geometry>
+    </collision>
+    <xacro:cylinder_inertia m="1.0" r="${camera_radius}" h="${camera_height}"/>
+  </link>
+  <!-- Camera link -->
+    <link name="camera_link">
+    <visual>
+      <origin xyz="0 ${camera_radius+camera_link_width/2.0} ${camera_link_length/2.0}" rpy="0 0 0"/>
+      <geometry>
+        <box size="${camera_link_depth} ${camera_link_width} ${camera_link_length}" />
+      </geometry>
+      <material name="white"/>
+    </visual>
+    <visual>
+      <origin xyz="0 -${camera_radius+camera_link_width/2.0} ${camera_link_length/2.0}" rpy="0 0 0"/>
+      <geometry>
+        <box size="${camera_link_depth} ${camera_link_width} ${camera_link_length}" />
+      </geometry>
+      <material name="white"/>
+    </visual>
+    <collision>
+      <origin xyz="0 ${camera_radius*2.0+camera_link_width/2.0} ${camera_link_length/2.0}" rpy="0 0 0"/>
+      <geometry>
+        <box size="${camera_link_depth} ${camera_link_width} ${camera_link_length}" />
+      </geometry>
+    </collision>
+    <xacro:box_inertia m="1.0" w="${camera_link_depth}" d="${camera_link_width}" h="${camera_link_length}"/>
+  </link>
   <!-- Camera joints -->
   <joint name="camera_sensor_joint" type="fixed">
     <origin xyz="${lens_length/2.0 + 0.1} 0 0" rpy="0 0 0"/>
     <parent link="camera_lens_link"/>
-    <child link="camera_link"/>
+    <child link="sensor_link"/>
   </joint>
   <joint name="camera_lens_joint" type="fixed">
-    <origin xyz="${camera_depth/2.0} 0 0" rpy="0 0 0"/>
+    <origin xyz="${3.0*camera_length/4.0} 0 0" rpy="0 0 0"/>
     <parent link="camera_body_link"/>
     <child link="camera_lens_link"/>
   </joint>
-  <joint name="camera_body_joint" type="fixed">
-    <origin xyz="${base_length/2.0 - camera_depth/2.0} 0 ${base_height/2.0 + camera_height/2.0}" rpy="0 0 0"/>
-    <parent link="base_link"/>
+  <joint name="camera_base_joint" type="revolute">
+    <origin xyz="${base_length/2.0-camera_radius*2.0} 0 ${base_height/2.0}" rpy="0 0 0"/>
+    <parent link="base_link"/>
+    <child link="camera_base"/>
+    <axis xyz="0 0 1" rpy="0 0 0"/>
+    <limit effort="30" velocity="1.0" lower="-31.415" upper="31.415" />
+  </joint>
+  <joint name="camera_link_joint" type="revolute">
+    <parent link="camera_base"/>
+    <child link="camera_link"/>
+    <origin xyz="0 0 ${camera_height-camera_offset}" rpy="0 0 0"/>
+    <axis xyz="0 1 0" rpy="0 0 0"/>
+    <limit effort="30" velocity="1.0" lower="-31.415" upper="31.415" />
+  </joint>
+  <joint name="camera_top_joint" type="revolute">
+    <parent link="camera_link"/>
     <child link="camera_body_link"/>
+    <origin xyz="0 0 ${camera_link_length-camera_offset}" rpy="0 0 0"/>
+    <axis xyz="0 1 0" rpy="0 0 0"/>
+    <limit effort="30" velocity="1.0" lower="-31.415" upper="31.415" />
   </joint>
   <!--                                       -->

File: smart_diffbot_description/model/urdf/utils.urdf.xacro (robot description, xacro)
@@ -20,4 +20,7 @@
     <color rgba="0 0 0 1"/>
   </material>
+  <material name="grey">
+    <color rgba="0.5 0.5 0.5 1"/>
+  </material>
   <!-- Inertia macros -->
   <xacro:macro name="box_inertia" params="m w h d">
@@ -33,4 +36,11 @@
       <mass value="${m}"/>
       <inertia ixx="${(m/12) * (3*r*r + h*h)}" ixy = "0" ixz = "0" iyy="${(m/12) * (3*r*r + h*h)}" iyz = "0" izz="${(m/2) * (r*r)}"/>
+    </inertial>
+  </xacro:macro>
+  <xacro:macro name="sphere_inertia" params="m r">
+    <inertial>
+      <origin xyz="0 0 0" rpy="0 0 0" />
+      <mass value="${m}"/>
+      <inertia ixx="${(2*m/5) * (r*r)}" ixy = "0" ixz = "0" iyy="${(2*m/5) * (r*r)}" iyz = "0" izz="${(2*m/5) * (r*r)}"/>
     </inertial>
   </xacro:macro>

Commit message: update model

File: smart_diffbot_description/model/urdf/model.urdf.xacro (robot description, xacro)
@@ -39,5 +39,5 @@
   <xacro:property name="camera_base_height" value="0.05"/>
   <xacro:property name="camera_offset" value="0.05"/>
-  <xacro:property name="camera_radius" value="0.075"/>
+  <xacro:property name="camera_radius" value="0.1"/>
   <xacro:property name="camera_link_length" value="0.3"/>
   <xacro:property name="lens_radius" value="0.04"/>

Commit message: move camera model to separate xacro

File: smart_diffbot_description/model/urdf/model.urdf.xacro (robot description, xacro)
@@ -1,4 +1,6 @@
 <?xml version="1.0"?>
 <robot xmlns:xacro="http://ros.org/wiki/xacro">
+  <!-- Camera model -->
+  <xacro:include filename="$(find smart_diffbot_description)/model/urdf/camera.urdf.xacro" />
   <!-- Properties -->
   <xacro:property name="base_length" value="1.5"/>
@@ -30,129 +32,6 @@
   </link>
   <link name="base_footprint"/>
-  <!--                                         -->
-  <!-- Start of camera on top of smart_diffbot -->
-  <!--                                         -->
-  <xacro:property name="camera_link_width" value="0.02"/>
-  <xacro:property name="camera_link_depth" value="0.05"/>
-  <xacro:property name="camera_length" value="0.25"/>
-  <xacro:property name="camera_height" value="0.1"/>
-  <xacro:property name="camera_base_height" value="0.05"/>
-  <xacro:property name="camera_offset" value="0.05"/>
-  <xacro:property name="camera_radius" value="0.1"/>
-  <xacro:property name="camera_link_length" value="0.3"/>
-  <xacro:property name="lens_radius" value="0.04"/>
-  <xacro:property name="lens_length" value="0.02"/>
-  <!-- Camera body -->
-  <link name="camera_body_link">
-    <visual>
-      <origin xyz="${camera_length/4} 0 0" rpy="0 ${pi/2} 0"/>
-      <geometry>
-        <cylinder radius="${camera_radius}" length="${camera_length}"/>
-      </geometry>
-      <material name="white" />
-    </visual>
-    <collision>
-      <origin xyz="0 0 0" rpy="0 0 0"/>
-      <geometry>
-        <cylinder radius="${camera_radius}" length="${camera_length}"/>
-      </geometry>
-    </collision>
-    <xacro:cylinder_inertia m="1.0" r="${camera_radius}" h="${camera_length}"/>
-  </link>
-  <!-- Camera lens -->
-  <link name="camera_lens_link">
-    <visual>
-      <origin xyz="0 0 0" rpy="0 ${pi/2} 0"/>
-      <geometry>
-        <cylinder radius="${lens_radius}" length="${lens_length}" />
-      </geometry>
-      <material name="black" />
-    </visual>
-    <collision>
-      <origin xyz="0 0 0" rpy="0 0 0"/>
-      <geometry>
-        <cylinder radius="${lens_radius}" length="${lens_length}" />
-      </geometry>
-    </collision>
-    <xacro:cylinder_inertia m="0.1" r="${lens_radius}" h="${lens_length}"/>
-  </link>
-  <!-- Camera sensor link -->
-  <link name="sensor_link"/>
-    <!-- Camera base -->
-  <link name="camera_base">
-    <visual>
-      <origin xyz="0 0 ${camera_base_height/2}" rpy="0 0 0"/>
-      <geometry>
-        <cylinder radius="${camera_radius}" length="${camera_height}" />
-      </geometry>
-      <material name="SaxionGreen" />
-    </visual>
-    <collision>
-      <origin xyz="0 0 ${camera_base_height/2}" rpy="0 0 0"/>
-      <geometry>
-        <cylinder radius="${camera_radius}" length="${camera_height}" />
-      </geometry>
-    </collision>
-    <xacro:cylinder_inertia m="1.0" r="${camera_radius}" h="${camera_height}"/>
-  </link>
-  <!-- Camera link -->
-    <link name="camera_link">
-    <visual>
-      <origin xyz="0 ${camera_radius+camera_link_width/2.0} ${camera_link_length/2.0}" rpy="0 0 0"/>
-      <geometry>
-        <box size="${camera_link_depth} ${camera_link_width} ${camera_link_length}" />
-      </geometry>
-      <material name="white"/>
-    </visual>
-    <visual>
-      <origin xyz="0 -${camera_radius+camera_link_width/2.0} ${camera_link_length/2.0}" rpy="0 0 0"/>
-      <geometry>
-        <box size="${camera_link_depth} ${camera_link_width} ${camera_link_length}" />
-      </geometry>
-      <material name="white"/>
-    </visual>
-    <collision>
-      <origin xyz="0 ${camera_radius*2.0+camera_link_width/2.0} ${camera_link_length/2.0}" rpy="0 0 0"/>
-      <geometry>
-        <box size="${camera_link_depth} ${camera_link_width} ${camera_link_length}" />
-      </geometry>
-    </collision>
-    <xacro:box_inertia m="1.0" w="${camera_link_depth}" d="${camera_link_width}" h="${camera_link_length}"/>
-  </link>
-  <!-- Camera joints -->
-  <joint name="camera_sensor_joint" type="fixed">
-    <origin xyz="${lens_length/2.0 + 0.1} 0 0" rpy="0 0 0"/>
-    <parent link="camera_lens_link"/>
-    <child link="sensor_link"/>
-  </joint>
-  <joint name="camera_lens_joint" type="fixed">
-    <origin xyz="${3.0*camera_length/4.0} 0 0" rpy="0 0 0"/>
-    <parent link="camera_body_link"/>
-    <child link="camera_lens_link"/>
-  </joint>
-  <joint name="camera_base_joint" type="revolute">
-    <origin xyz="${base_length/2.0-camera_radius*2.0} 0 ${base_height/2.0}" rpy="0 0 0"/>
-    <parent link="base_link"/>
-    <child link="camera_base"/>
-    <axis xyz="0 0 1" rpy="0 0 0"/>
-    <limit effort="30" velocity="1.0" lower="-31.415" upper="31.415" />
-  </joint>
-  <joint name="camera_link_joint" type="revolute">
-    <parent link="camera_base"/>
-    <child link="camera_link"/>
-    <origin xyz="0 0 ${camera_height-camera_offset}" rpy="0 0 0"/>
-    <axis xyz="0 1 0" rpy="0 0 0"/>
-    <limit effort="30" velocity="1.0" lower="-31.415" upper="31.415" />
-  </joint>
-  <joint name="camera_top_joint" type="revolute">
-    <parent link="camera_link"/>
-    <child link="camera_body_link"/>
-    <origin xyz="0 0 ${camera_link_length-camera_offset}" rpy="0 0 0"/>
-    <axis xyz="0 1 0" rpy="0 0 0"/>
-    <limit effort="30" velocity="1.0" lower="-31.415" upper="31.415" />
-  </joint>
-  <!--                                       -->
-  <!-- End of camera on top of smart_diffbot -->
-  <!--                                       -->
+  <link name="camera_mount"/>
+  <xacro:camera name="camera" parent="camera_mount"/>
   <!-- Other sensor links (not visualized) -->
   <link name="imu_link"/>
@@ -182,4 +61,9 @@
       <parent link="base_link"/>
       <child link="base_footprint"/>
+  </joint>
+  <joint name="camera_mount_joint" type="fixed">
+    <origin xyz="${base_length/2.0-camera_radius*2.0} 0 ${base_height/2.0}" rpy="0 0 0"/>
+    <parent link="base_link"/>
+    <child link="camera_mount"/>
   </joint>
   <joint name="imu_joint" type="fixed">
