Commit message: update model with articulated camera

File: smart_diffbot_description/model/urdf/model.urdf.xacro (robot description, xacro)
@@ -1,4 +1,6 @@
 <?xml version="1.0"?>
 <robot xmlns:xacro="http://ros.org/wiki/xacro">
+  <!-- Camera model -->
+  <xacro:include filename="$(find smart_diffbot_description)/model/urdf/camera.urdf.xacro" />
   <!-- Properties -->
   <xacro:property name="base_length" value="0.1415"/>
@@ -9,5 +11,5 @@
   <xacro:property name="wheel_suspension" value="0.01"/>
   <xacro:property name="wheel_spacing" value="0.002"/>
-  <xacro:property name="caster_radius" value="0.01"/>
+  <xacro:property name="caster_radius" value="0.015"/>
   <!-- Links -->
   <link name="base_link">
@@ -30,67 +32,6 @@
   </link>
   <link name="base_footprint"/>
-  <!--                                         -->
-  <!-- Start of camera on top of smart_diffbot -->
-  <!--                                         -->
-  <xacro:property name="camera_width" value="0.02"/>
-  <xacro:property name="camera_depth" value="0.005"/>
-  <xacro:property name="camera_height" value="0.01"/>
-  <xacro:property name="lens_radius" value="0.003"/>
-  <xacro:property name="lens_length" value="0.002"/>
-  <!-- Camera body -->
-  <link name="camera_body_link">
-    <visual>
-      <origin xyz="0 0 0" rpy="0 0 0"/>
-      <geometry>
-        <box size="${camera_depth} ${camera_width} ${camera_height}" />
-      </geometry>
-      <material name="black" />
-    </visual>
-    <collision>
-      <origin xyz="0 0 0" rpy="0 0 0"/>
-      <geometry>
-        <box size="${camera_depth} ${camera_width} ${camera_height}" />
-      </geometry>
-    </collision>
-    <xacro:box_inertia m="1.0" w="${camera_width}" d="${camera_depth}" h="${camera_height}"/>
-  </link>
-  <!-- Camera lens -->
-  <link name="camera_lens_link">
-    <visual>
-      <origin xyz="0 0 0" rpy="0 ${pi/2} 0"/>
-      <geometry>
-        <cylinder radius="${lens_radius}" length="${lens_length}" />
-      </geometry>
-      <material name="white" />
-    </visual>
-    <collision>
-      <origin xyz="0 0 0" rpy="0 0 0"/>
-      <geometry>
-        <cylinder radius="${lens_radius}" length="${lens_length}" />
-      </geometry>
-    </collision>
-    <xacro:cylinder_inertia m="0.1" r="${lens_radius}" h="${lens_length}"/>
-  </link>
-  <!-- Camera sensor link -->
-  <link name="camera_link"/>
-  <!-- Camera joints -->
-  <joint name="camera_sensor_joint" type="fixed">
-    <origin xyz="${lens_length/2.0 + 0.1} 0 0" rpy="0 0 0"/>
-    <parent link="camera_lens_link"/>
-    <child link="camera_link"/>
-  </joint>
-  <joint name="camera_lens_joint" type="fixed">
-    <origin xyz="${camera_depth/2.0} 0 0" rpy="0 0 0"/>
-    <parent link="camera_body_link"/>
-    <child link="camera_lens_link"/>
-  </joint>
-  <joint name="camera_body_joint" type="fixed">
-    <origin xyz="${base_length/2.0 - camera_depth/2.0} 0 ${base_height/2.0 + camera_height/2.0}" rpy="0 0 0"/>
-    <parent link="base_link"/>
-    <child link="camera_body_link"/>
-  </joint>
-  <!--                                       -->
-  <!-- End of camera on top of smart_diffbot -->
-  <!--                                       -->
+  <link name="camera_mount"/>
+  <xacro:camera name="camera" parent="camera_mount"/>
   <!-- Other sensor links (not visualized) -->
   <link name="imu_link"/>
@@ -113,5 +54,5 @@
       </geometry>
     </collision>
-    <xacro:box_inertia m="0.5" w="${base_width}" d="${base_length}" h="${base_height}"/>
+    <xacro:sphere_inertia m="0.25" r="${caster_radius}"/>
   </link>
   <!-- Joints -->
@@ -120,4 +61,9 @@
       <parent link="base_link"/>
       <child link="base_footprint"/>
+  </joint>
+  <joint name="camera_mount_joint" type="fixed">
+    <origin xyz="${base_length/2.0-camera_radius*2.0} 0 ${base_height/2.0}" rpy="0 0 0"/>
+    <parent link="base_link"/>
+    <child link="camera_mount"/>
   </joint>
   <joint name="imu_joint" type="fixed">

Commit message: fix model

File: smart_diffbot_description/model/urdf/model.urdf.xacro (robot description, xacro)
@@ -56,9 +56,4 @@
   </link>
   <!-- Joints -->
-  <joint name="footprint_joint" type="fixed">
-      <origin xyz="0 0 ${- base_height/2.0 - wheel_radius + wheel_suspension}" rpy="0 0 0"/>
-      <parent link="base_link"/>
-      <child link="base_footprint"/>
-  </joint>
   <joint name="camera_mount_joint" type="fixed">
     <origin xyz="${base_length/2.0-camera_radius*2.0} 0 ${base_height/2.0}" rpy="0 0 0"/>
